File: pcb/switch/switch.kicad_sch (KiCad schematic)
At the start: 29 parts, among them J1 Conn_01x06, J2 Conn_01x04, J3 Conn_01x05, J4 Conn_01x04, K1 G6SU-2, K2 G6SU-2, K3 G6SU-2, K4 G6SU-2, SW1 D2F-01, SW2 D2F-01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

Commit message: Port symbol library to KiCad 6
Connections:
- net GND: now also U3.9 (EP)
Changed lines of the file:
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@@
   (junction (at 45.72 58.42) (diameter 0) (color 0 0 0 0)
+  )
+  (junction (at 77.47 140.97) (diameter 0) (color 0 0 0 0)
   )
   (junction (at 54.61 123.19) (diameter 0) (color 0 0 0 0)
@@
     (stroke (width 0) (type default) (color 0 0 0 0))
   )
+  (wire (pts (xy 74.93 140.97) (xy 77.47 140.97))
+    (stroke (width 0) (type default) (color 0 0 0 0))
+  )
   (wire (pts (xy 218.44 133.35) (xy 218.44 135.89))
     (stroke (width 0) (type default) (color 0 0 0 0))
@@
   )
   (wire (pts (xy 86.36 123.19) (xy 97.79 123.19))
-    (stroke (width 0) (type default) (color 0 0 0 0))
-  )
-  (wire (pts (xy 74.93 140.97) (xy 97.79 140.97))
     (stroke (width 0) (type default) (color 0 0 0 0))
   )
@@
     (stroke (width 0) (type default) (color 0 0 0 0))
   )
+  (wire (pts (xy 77.47 140.97) (xy 97.79 140.97))
+    (stroke (width 0) (type default) (color 0 0 0 0))
+  )
