File: pcb/control/control.kicad_sch (KiCad schematic)
At the start: 79 parts, among them J1 Conn_01x06, J10 Conn_01x02, J2 Conn_01x05, J3 Conn_01x01, J4 USB_B_Micro, J5 Conn_01x04, J6 Conn_01x06, J7 Conn_01x02, J8 Conn_01x02, J9 Conn_01x01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

Commit message: Port symbol library to KiCad 6
Parts:
- U11: footprint RoomControl:MR45V064B -> RoomControl:FM25CL64B
- gave numbers to parts that had none: 1
Changed lines of the file:
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@@
   (junction (at 41.91 104.14) (diameter 0) (color 0 0 0 0)
   )
-  (junction (at 177.8 41.91) (diameter 0) (color 0 0 0 0)
-  )
   (junction (at 157.48 24.13) (diameter 0) (color 0 0 0 0)
   )
@@
   (junction (at 323.85 100.33) (diameter 0) (color 0 0 0 0)
   )
+  (junction (at 177.8 41.91) (diameter 0) (color 0 0 0 0)
+  )
   (junction (at 41.91 124.46) (diameter 0) (color 0 0 0 0)
   )
@@
     (stroke (width 0) (type default) (color 0 0 0 0))
   )
-  (wire (pts (xy 180.34 41.91) (xy 177.8 41.91))
-    (stroke (width 0) (type default) (color 0 0 0 0))
-  )
   (wire (pts (xy 148.59 95.25) (xy 148.59 90.17))
     (stroke (width 0) (type default) (color 0 0 0 0))
@@
     (stroke (width 0) (type default) (color 0 0 0 0))
   )
+  (wire (pts (xy 177.8 41.91) (xy 180.34 41.91))
+    (stroke (width 0) (type default) (color 0 0 0 0))
+  )
   (wire (pts (xy 275.59 96.52) (xy 275.59 104.14))
     (stroke (width 0) (type default) (color 0 0 0 0))
@@
   (symbol (lib_id "Jumper:SolderJumper_2_Open") (at 140.97 105.41 90) (unit 1)
     (in_bom yes) (on_board yes)
-    (property "Reference" "" (id 0) (at 138.43 105.41 0))
+    (property "Reference" "JP10" (id 0) (at 138.43 105.41 0))
     (property "Value" "SolderJumper_2_Open" (id 1) (at 127 97.79 0))
     (property "Footprint" "RoomControl:Jumper2" (id 2) (at 140.97 105.41 0)
@@
     (property "Reference" "U11" (id 0) (at 194.31 62.23 0))
     (property "Value" "FM25CL64B" (id 1) (at 207.01 62.23 0))
-    (property "Footprint" "RoomControl:MR45V064B" (id 2) (at 200.66 71.12 0)
+    (property "Footprint" "RoomControl:FM25CL64B" (id 2) (at 200.66 71.12 0)
       (effects (font (size 1.27 1.27)) hide)
     )
@@
     )
     (path "/00000000-0000-0000-0000-000060793bb9"
-      (reference "U11") (unit 1) (value "FM25CL64B") (footprint "RoomControl:MR45V064B")
+      (reference "U11") (unit 1) (value "FM25CL64B") (footprint "RoomControl:FM25CL64B")
     )
     (path "/00000000-0000-0000-0000-00006069a51b"

Commit message: Minor fixes
Connections:
- net GND: now also U9.25 (PAD)
Changed lines of the file:
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@@
   (junction (at 118.11 33.02) (diameter 0) (color 0 0 0 0)
   )
+  (junction (at 111.76 119.38) (diameter 0) (color 0 0 0 0)
+  )
+  (junction (at 143.51 97.79) (diameter 0) (color 0 0 0 0)
+  )
+  (junction (at 330.2 85.09) (diameter 0) (color 0 0 0 0)
+  )
+  (junction (at 118.11 40.64) (diameter 0) (color 0 0 0 0)
+  )
+  (junction (at 257.81 104.14) (diameter 0) (color 0 0 0 0)
+  )
+  (junction (at 41.91 88.9) (diameter 0) (color 0 0 0 0)
+  )
+  (junction (at 118.11 25.4) (diameter 0) (color 0 0 0 0)
+  )
+  (junction (at 140.97 97.79) (diameter 0) (color 0 0 0 0)
+  )
+  (junction (at 101.6 40.64) (diameter 0) (color 0 0 0 0)
+  )
+  (junction (at 323.85 100.33) (diameter 0) (color 0 0 0 0)
+  )
+  (junction (at 177.8 41.91) (diameter 0) (color 0 0 0 0)
+  )
+  (junction (at 41.91 124.46) (diameter 0) (color 0 0 0 0)
+  )
+  (junction (at 336.55 85.09) (diameter 0) (color 0 0 0 0)
+  )
+  (junction (at 275.59 119.38) (diameter 0) (color 0 0 0 0)
+  )
+  (junction (at 104.14 124.46) (diameter 0) (color 0 0 0 0)
+  )
+  (junction (at 111.76 124.46) (diameter 0) (color 0 0 0 0)
+  )
+  (junction (at 41.91 81.28) (diameter 0) (color 0 0 0 0)
+  )
+  (junction (at 90.17 25.4) (diameter 0) (color 0 0 0 0)
+  )
+  (junction (at 317.5 100.33) (diameter 0) (color 0 0 0 0)
+  )
+  (junction (at 148.59 90.17) (diameter 0) (color 0 0 0 0)
+  )
+  (junction (at 363.22 85.09) (diameter 0) (color 0 0 0 0)
+  )
+  (junction (at 142.24 172.72) (diameter 0) (color 0 0 0 0)
+  )
+  (junction (at 157.48 31.75) (diameter 0) (color 0 0 0 0)
+  )
+  (junction (at 30.48 140.97) (diameter 0) (color 0 0 0 0)
+  )
+  (junction (at 212.09 69.85) (diameter 0) (color 0 0 0 0)
+  )
+  (junction (at 35.56 160.02) (diameter 0) (color 0 0 0 0)
+  )
+  (junction (at 232.41 114.3) (diameter 0) (color 0 0 0 0)
+  )
+  (junction (at 41.91 121.92) (diameter 0) (color 0 0 0 0)
+  )
+  (junction (at 82.55 25.4) (diameter 0) (color 0 0 0 0)
+  )
+  (junction (at 248.92 116.84) (diameter 0) (color 0 0 0 0)
+  )
+  (junction (at 38.1 26.67) (diameter 0) (color 0 0 0 0)
+  )
+  (junction (at 241.3 116.84) (diameter 0) (color 0 0 0 0)
+  )
+  (junction (at 257.81 96.52) (diameter 0) (color 0 0 0 0)
+  )
+  (junction (at 41.91 91.44) (diameter 0) (color 0 0 0 0)
+  )
+  (junction (at 41.91 114.3) (diameter 0) (color 0 0 0 0)
+  )
+  (junction (at 38.1 190.5) (diameter 0) (color 0 0 0 0)
+  )
+  (junction (at 252.73 64.77) (diameter 0) (color 0 0 0 0)
+  )
+  (junction (at 275.59 104.14) (diameter 0) (color 0 0 0 0)
+  )
   (junction (at 36.83 140.97) (diameter 0) (color 0 0 0 0)
   )
-  (junction (at 111.76 119.38) (diameter 0) (color 0 0 0 0)
-  )
-  (junction (at 143.51 97.79) (diameter 0) (color 0 0 0 0)
-  )
-  (junction (at 330.2 85.09) (diameter 0) (color 0 0 0 0)
-  )
-  (junction (at 118.11 40.64) (diameter 0) (color 0 0 0 0)
-  )
-  (junction (at 257.81 104.14) (diameter 0) (color 0 0 0 0)
-  )
-  (junction (at 41.91 88.9) (diameter 0) (color 0 0 0 0)
-  )
-  (junction (at 118.11 25.4) (diameter 0) (color 0 0 0 0)
-  )
-  (junction (at 140.97 97.79) (diameter 0) (color 0 0 0 0)
-  )
-  (junction (at 101.6 40.64) (diameter 0) (color 0 0 0 0)
-  )
-  (junction (at 323.85 100.33) (diameter 0) (color 0 0 0 0)
-  )
-  (junction (at 177.8 41.91) (diameter 0) (color 0 0 0 0)
-  )
-  (junction (at 41.91 124.46) (diameter 0) (color 0 0 0 0)
-  )
-  (junction (at 336.55 85.09) (diameter 0) (color 0 0 0 0)
-  )
-  (junction (at 275.59 119.38) (diameter 0) (color 0 0 0 0)
-  )
-  (junction (at 104.14 124.46) (diameter 0) (color 0 0 0 0)
-  )
-  (junction (at 111.76 124.46) (diameter 0) (color 0 0 0 0)
-  )
-  (junction (at 41.91 81.28) (diameter 0) (color 0 0 0 0)
-  )
-  (junction (at 90.17 25.4) (diameter 0) (color 0 0 0 0)
-  )
-  (junction (at 317.5 100.33) (diameter 0) (color 0 0 0 0)
-  )
-  (junction (at 148.59 90.17) (diameter 0) (color 0 0 0 0)
-  )
-  (junction (at 363.22 85.09) (diameter 0) (color 0 0 0 0)
-  )
-  (junction (at 142.24 172.72) (diameter 0) (color 0 0 0 0)
-  )
-  (junction (at 157.48 31.75) (diameter 0) (color 0 0 0 0)
-  )
-  (junction (at 212.09 69.85) (diameter 0) (color 0 0 0 0)
-  )
-  (junction (at 35.56 160.02) (diameter 0) (color 0 0 0 0)
-  )
-  (junction (at 232.41 114.3) (diameter 0) (color 0 0 0 0)
-  )
-  (junction (at 41.91 121.92) (diameter 0) (color 0 0 0 0)
-  )
-  (junction (at 82.55 25.4) (diameter 0) (color 0 0 0 0)
-  )
-  (junction (at 248.92 116.84) (diameter 0) (color 0 0 0 0)
-  )
-  (junction (at 38.1 26.67) (diameter 0) (color 0 0 0 0)
-  )
-  (junction (at 241.3 116.84) (diameter 0) (color 0 0 0 0)
-  )
-  (junction (at 257.81 96.52) (diameter 0) (color 0 0 0 0)
-  )
-  (junction (at 41.91 91.44) (diameter 0) (color 0 0 0 0)
-  )
-  (junction (at 41.91 114.3) (diameter 0) (color 0 0 0 0)
-  )
-  (junction (at 38.1 190.5) (diameter 0) (color 0 0 0 0)
-  )
-  (junction (at 252.73 64.77) (diameter 0) (color 0 0 0 0)
-  )
-  (junction (at 275.59 104.14) (diameter 0) (color 0 0 0 0)
-  )
   (junction (at 41.91 116.84) (diameter 0) (color 0 0 0 0)
   )
@@
     (stroke (width 0) (type default) (color 0 0 0 0))
   )
+  (wire (pts (xy 27.94 140.97) (xy 30.48 140.97))
+    (stroke (width 0) (type default) (color 0 0 0 0))
+  )
   (wire (pts (xy 363.22 100.33) (xy 379.73 100.33))
     (stroke (width 0) (type default) (color 0 0 0 0))
@@
     (stroke (width 0) (type default) (color 0 0 0 0))
   )
+  (wire (pts (xy 30.48 140.97) (xy 36.83 140.97))
+    (stroke (width 0) (type default) (color 0 0 0 0))
+  )
   (wire (pts (xy 46.99 129.54) (xy 46.99 133.35))
     (stroke (width 0) (type default) (color 0 0 0 0))
@@
     (stroke (width 0) (type default) (color 0 0 0 0))
   )
-  (wire (pts (xy 27.94 140.97) (xy 36.83 140.97))
-    (stroke (width 0) (type default) (color 0 0 0 0))
-  )
